File: PDM/PDM.kicad_pcb (KiCad board)
At the start: 4 copper layers, 124 x 116 mm, 224 parts, among them J1 HCCPHPE24BKA90F, J2 M6 VBAT, Q1 BSS84, Q2 BSP75N, U1 LM2937IMP-5.0, U10 BTS7002-1EPP, U11 BTS7002-1EPP, U12 BTS7002-1EPP, U13 BTS7002-1EPP, U14 BTS7002-1EPP, U15 BTS7002-1EPP, U16 BTS7002-1EPP, U17 BTS7002-1EPP, U3 74HC86-Q100, U4 74HC86-Q100, U5 LM2901AVQDR (-Q1), U6 LM2901AVQDR (-Q1), U7 LM2901AVQDR (-Q1), U8 LM2901AVQDR (-Q1), U9 LM2901AVQDR (-Q1)

Commit message: PDM: manufacturer part numbers, order list and fabrication outputs
- Manufacturer + MPN fields on all 220 symbols and footprints
  (tools/parts.py, automotive grade where available; C2 22u -> 47u/50V,
  same part as C1); ERC 0, DRC 0 errors, 0 parity issues
- BOM.csv with Manufacturer/MPN columns
- docs/PDM_objednavka.xlsx (tools/order_xlsx.py): order list grouped by
  MPN with board count / spare inputs, PCB fab parameters, mechanics
- fab/: Gerber X2 + Excellon drill (PDM_gerber.zip), placement CSV

Co-Authored-By: Claude Opus 5.5 <noreply@anthropic.com>
Claude-Session: https://claude.ai/code/session_011RdW2Ae3jMjzHoNbLtu1MC
Parts:
- C2: value 22u/50V -> 47u/50V
