File: PDM/PDM.kicad_sch (KiCad schematic)
At the start: 225 parts, among them J1 HCCPHPE24BKA90F, J2 M6 VBAT, Q1 BSS84, Q2 BSP75N, U1 LM2937IMP-5.0, U10 BTS7002-1EPP, U11 BTS7002-1EPP, U12 BTS7002-1EPP, U13 BTS7002-1EPP, U14 BTS7002-1EPP, U15 BTS7002-1EPP, U16 BTS7002-1EPP, U17 BTS7002-1EPP, U2 LMR36520ADDAR, U3 74HC86-Q100, U4 74HC86-Q100, U5 LM2901AVQDR (-Q1), U6 LM2901AVQDR (-Q1), U7 LM2901AVQDR (-Q1), U8 LM2901AVQDR (-Q1), U9 LM2901AVQDR (-Q1)

Commit message: PDM schematic: 12V display output, clamped comparator supply, +5V back-feed fix
Verified against the BTS7002-1EPP datasheet (kILIS 22900, IIS(FAULT) >= 4.4 mA,
VS 28 V / 35 V suppressed load dump, pin 5-7 and 11 n.c., DZ2 33 V TVS).

- 5V display buck (U2, L1, C6, C7, C9-C12, R1, R2) removed; J1 C6 is now
  +12V_DISP = VKEY through F1 0.5 A PTC, 5 V made externally
- VCOMP: VKEY -> R96 470R -> D45 18 V zener, supplies U5-U9, R19, R23 and
  Q1 source (LM2901 36 V max, BSS84 VGS 20 V max at jump start/load dump)
- R17/R18 6k81/10k -> 68k1/100k (same 2.97 V REF_FLT) and R97 1k minimum
  load on +5V: LM2937 cannot sink the current fed back via REF_FLT and the
  input clamps
- R23 4k7 -> 22k (VCOMP current), C23 220n -> 330n (~2.2 Hz blink)
- tools/sch_edit.py: editor used for the changes; BOM.csv regenerated
- PCB not updated yet (re-route in progress)

Co-Authored-By: Claude Opus 5.5 <noreply@anthropic.com>
Claude-Session: https://claude.ai/code/session_011RdW2Ae3jMjzHoNbLtu1MC
Parts:
- removed C10: 1u/16V, Capacitor_SMD:C_0805_2012Metric, symbol PDM:C
- removed C11, C12: 22u/25V, Capacitor_SMD:C_1210_3225Metric, symbol PDM:C
- removed C6, C7: 4u7/100V, Capacitor_SMD:C_1210_3225Metric, symbol PDM:C
- removed C9: 100n/16V, Capacitor_SMD:C_0805_2012Metric, symbol PDM:C
- removed L1: 10u Isat>=3.6A, Inductor_SMD:L_Bourns_SRP7028A_7.3x6.6mm, symbol PDM:L
- removed R1: 100k 1%, Resistor_SMD:R_0805_2012Metric, symbol PDM:R
- removed R2: 24k9 1%, Resistor_SMD:R_0805_2012Metric, symbol PDM:R
- removed U2: LMR36520ADDAR, Package_SO:TI_SO-PowerPAD-8_ThermalVias, symbol PDM:LMR36520
- added C62: 1u/50V, Capacitor_SMD:C_0805_2012Metric, symbol PDM:C
- added D45: 18V 1W SMAZ18, Diode_SMD:D_SMA, symbol PDM:D_Zener
- added F1: 0.5A PTC 1812L050/33, Fuse:Fuse_1812_4532Metric, symbol PDM:Polyfuse
- added R96: 470R, Resistor_SMD:R_1206_3216Metric, symbol PDM:R
- added R97: 1k, Resistor_SMD:R_0805_2012Metric, symbol PDM:R
- C23: value 220n -> 330n
- R17: value 6k81 1% -> 68k1 1%
- R18: value 10k 1% -> 100k 1%
- R23: value 4k7 -> 22k
Connections:
- net +5V: now also R97.1
- net GND: now also C62.2, D45.2 (A), R97.2
- net VKEY: now also F1.1, R96.1; no longer C25.1, C26.1, C27.1, C28.1, C29.1, Q1.2 (S), R19.1, R23.1, U5.3 (VCC), U6.3 (VCC), U7.3 (VCC), U8.3 (VCC), U9.3 (VCC)
- net +5V_DISP renamed +12V_DISP
- net +12V_DISP: now also F1.2
- new net VCOMP: C25.1, C26.1, C27.1, C28.1, C29.1, C62.1, D45.1 (K), Q1.2 (S), R19.1, R23.1, R96.2, U5.3 (VCC), U6.3 (VCC), U7.3 (VCC), U8.3 (VCC), U9.3 (VCC)
Other:
- note added: "12V DISPLAY 0.5A (PTC) / VCOMP 18V"
- note removed: "5V DISPLAY 2A"

Commit message: PDM: manufacturer part numbers, order list and fabrication outputs
- Manufacturer + MPN fields on all 220 symbols and footprints
  (tools/parts.py, automotive grade where available; C2 22u -> 47u/50V,
  same part as C1); ERC 0, DRC 0 errors, 0 parity issues
- BOM.csv with Manufacturer/MPN columns
- docs/PDM_objednavka.xlsx (tools/order_xlsx.py): order list grouped by
  MPN with board count / spare inputs, PCB fab parameters, mechanics
- fab/: Gerber X2 + Excellon drill (PDM_gerber.zip), placement CSV

Co-Authored-By: Claude Opus 5.5 <noreply@anthropic.com>
Claude-Session: https://claude.ai/code/session_011RdW2Ae3jMjzHoNbLtu1MC
Parts:
- C1: MPN (none) -> EEE-FK1H470P; Manufacturer (none) -> Panasonic
- C13, C14, C15, C16, C17, C22, C32, C36, C40, C44, C48, C52, C56, C60: MPN (none) -> CL21B103KBANNNC; Manufacturer (none) -> Samsung
- C18, C19, C20, C21, C25, C26, C27, C28, C29, C3, C31, C35, C39, C43, C47, C5, C51, C55, C59: MPN (none) -> CL21B104KBCNNNC; Manufacturer (none) -> Samsung
- C2: value 22u/50V -> 47u/50V; MPN (none) -> EEE-FK1H470P; Manufacturer (none) -> Panasonic
- C23: MPN (none) -> CL21B334KBFNNNE; Manufacturer (none) -> Samsung
- C24, C33, C37, C41, C45, C49, C53, C57, C61: MPN (none) -> CL21A106KOQNNNE; Manufacturer (none) -> Samsung
- C30, C34, C38, C42, C46, C50, C54, C58: MPN (none) -> CL21B473KBANNNC; Manufacturer (none) -> Samsung
- C4: MPN (none) -> T491B226K010AT; Manufacturer (none) -> KEMET
- C62: MPN (none) -> CL21B105KBFNNNE; Manufacturer (none) -> Samsung
- C8: MPN (none) -> GCM21BR72A224KA37L; Manufacturer (none) -> Murata
- D1: MPN (none) -> SMCJ33A; Manufacturer (none) -> Littelfuse
- D10, D11, D12, D15, D16, D19, D20, D23, D24, D27, D28, D31, D32, D35, D36, D39, D40, D43, D44, D9: MPN (none) -> BAT54,215; Manufacturer (none) -> Nexperia
- D13, D17, D21, D25, D29, D33, D37, D41: MPN (none) -> 150080GS75000; Manufacturer (none) -> Wurth Elektronik
- D14, D18, D22, D26, D30, D34, D38, D42: MPN (none) -> 150080RS75000; Manufacturer (none) -> Wurth Elektronik
- D2: MPN (none) -> SS34-E3/61T; Manufacturer (none) -> Vishay
- D3: MPN (none) -> SMBJ33A; Manufacturer (none) -> Littelfuse
- D4, D5, D6, D7, D8: MPN (none) -> BAV99,215; Manufacturer (none) -> Nexperia
- D45: MPN (none) -> SMAZ18-13-F; Manufacturer (none) -> Diodes Inc.
- F1: MPN (none) -> 1812L050/33MR; Manufacturer (none) -> Littelfuse
- J1: MPN (none) -> HCCPHPE24BKA90F; Manufacturer (none) -> Amphenol FCI
- J2: MPN (none) -> -; Manufacturer (none) -> -
- JP1, JP2, JP3: MPN (none) -> 61300311121; Manufacturer (none) -> Wurth Elektronik
- Q1: MPN (none) -> BSS84,215; Manufacturer (none) -> Nexperia
- Q2: MPN (none) -> BSP75NH6327XTSA1; Manufacturer (none) -> Infineon
- R10, R12, R4, R6, R8: MPN (none) -> RC0805FR-0747KL; Manufacturer (none) -> Yageo
- R11, R14, R16, R25, R26, R27, R28, R29, R3, R36, R39, R44, R47, R5, R52, R55, R60, R63, R68, R7, R71, R76, R79, R84, R87, R9, R92, R95: MPN (none) -> RC0805FR-0710KL; Manufacturer (none) -> Yageo
- R13: MPN (none) -> RC0805FR-0735K7L; Manufacturer (none) -> Yageo
- R15: MPN (none) -> RC0805FR-0766K5L; Manufacturer (none) -> Yageo
- R17: MPN (none) -> RC0805FR-0768K1L; Manufacturer (none) -> Yageo
- R18, R19, R20, R21, R31: MPN (none) -> RC0805FR-07100KL; Manufacturer (none) -> Yageo
- R22: MPN (none) -> RC0805FR-071ML; Manufacturer (none) -> Yageo
- R23: MPN (none) -> RC0805FR-0722KL; Manufacturer (none) -> Yageo
- R24: MPN (none) -> RC0805FR-07300KL; Manufacturer (none) -> Yageo
- R30, R32, R33, R40, R41, R48, R49, R56, R57, R64, R65, R72, R73, R80, R81, R88, R89: MPN (none) -> RC0805FR-074K7L; Manufacturer (none) -> Yageo
- R34, R42, R50, R58, R66, R74, R82, R90: MPN (none) -> RC0805FR-0747RL; Manufacturer (none) -> Yageo
- R35, R38, R43, R46, R51, R54, R59, R62, R67, R70, R75, R78, R83, R86, R91, R94, R97: MPN (none) -> RC0805FR-071KL; Manufacturer (none) -> Yageo
- R37, R45, R53, R61, R69, R77, R85, R93: MPN (none) -> RC0805FR-073K9L; Manufacturer (none) -> Yageo
- R96: MPN (none) -> RC1206FR-07470RL; Manufacturer (none) -> Yageo
- U1: MPN (none) -> LM2937IMP-5.0/NOPB; Manufacturer (none) -> Texas Instruments
- U10, U11, U12, U13, U14, U15, U16, U17: MPN (none) -> BTS70021EPPXUMA1; Manufacturer (none) -> Infineon
- U3, U4: MPN (none) -> 74HC86D-Q100J; Manufacturer (none) -> Nexperia
- U5, U6, U7, U8, U9: MPN (none) -> LM2901AVQDRQ1; Manufacturer (none) -> Texas Instruments
