File: dash/notstock-can185/notstock-can185.kicad_pcb (KiCad board)
At the start: 2 copper layers, 48 x 48 mm, 31 parts, among them J1 OBD 12V GND H L 15, J2 UART wires from display, J3 BAT to display, U1 LMR16006YDDCR, U2 SN65HVD230

Commit message: CAN 1.85 rev 6: 12 V from OBD pin 1 (terminal 15), 4-pin J1 again
The board takes its supply from the key-switched pin 1 instead of the
permanent pin 16, so the ignition input and its divider are not needed.

Co-Authored-By: Claude Opus 5.5 <noreply@anthropic.com>
Claude-Session: https://claude.ai/code/session_018SKN4tJhAPpVCWtvRZgZpD
Parts:
- removed C9: 100n, Capacitor_SMD:C_0603_1608Metric
- removed R9: 13k, Resistor_SMD:R_0603_1608Metric
- J1: value OBD 12V GND H L 15 -> OBD 12V GND H L; footprint Connector_JST:JST_PH_B5B-PH-SM4-TB_1x05-1MP_P2.00mm_Vertical -> Connector_JST:JST_PH_B4B-PH-SM4-TB_1x04-1MP_P2.00mm_Vertical
- moved J1 1.00 mm to (152.0, 84.5)
Connections:
- R1 pad 1: IGN -> VIN
Routing:
- net IGN: track 36.8 -> 0.00 mm
- net GND: track 179.0 -> 157.8 mm, vias 66 -> 77
- net CANH: track 49.9 -> 35.3 mm
- net EN: track 13.9 -> 2.54 mm
- net BAT_LCD: track 41.0 -> 30.4 mm, vias 1 -> 0
- net CANL: track 32.5 -> 40.9 mm
- net +3V3: track 58.7 -> 50.9 mm
- net TMID: track 15.6 -> 18.9 mm, vias 0 -> 2
- net VIN: track 23.1 -> 25.3 mm
Other:
- board text added: "rev 6"
- board text removed: "15"
- board text removed: "rev 5"

Commit message: CAN boards: D3 K16 (C2943756) for the PMEG6010CEH out of stock
Same footprint (SOD-123FL on the SOD-123F pads), 60 V 1 A Schottky.
BOM, schematic and the boards' LCSC fields updated on both boards.

Co-Authored-By: Claude Opus 5.5 <noreply@anthropic.com>
Claude-Session: https://claude.ai/code/session_018SKN4tJhAPpVCWtvRZgZpD
Parts:
- D3: value PMEG6010CEH -> K16
Changed lines of the file:
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@@
     (descr "D_SOD-123F")
     (tags "D_SOD-123F")
-    (property "LCSC" "C110797")
+    (property "LCSC" "C2943756")
     (attr smd)
     (fp_text reference "D3" (at -0.0225 -1.875 180) (layer "F.SilkS")
         (effects (font (size 0.8 0.8) (thickness 0.13)))
     )
-    (fp_text value "PMEG6010CEH" (at 0 2.1 180) (layer "F.Fab") hide
+    (fp_text value "K16" (at 0 2.1 180) (layer "F.Fab") hide
         (effects (font (size 1 1) (thickness 0.15)))
     )

Commit message: CAN boards: JLCPCB basic parts where possible
D1 SS16 -> SS34 (C8678, basic, same SMA footprint) on both boards.
CAN 1.32: C4/C5 22 uF 1206 -> 0805 25 V (C45783, basic), rerouted,
DRC clean.

Co-Authored-By: Claude Opus 5.5 <noreply@anthropic.com>
Claude-Session: https://claude.ai/code/session_018SKN4tJhAPpVCWtvRZgZpD
Parts:
- D1: value SS16 -> SS34
Changed lines of the file:
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@@
     (descr "Diode SMA (DO-214AC)")
     (tags "Diode SMA (DO-214AC)")
-    (property "LCSC" "C2758574")
+    (property "LCSC" "C8678")
     (attr smd)
     (fp_text reference "D1" (at 4.225001 0 90) (layer "F.SilkS")
         (effects (font (size 0.8 0.8) (thickness 0.13)))
     )
-    (fp_text value "SS16" (at 0 2.6 90) (layer "F.Fab") hide
+    (fp_text value "SS34" (at 0 2.6 90) (layer "F.Fab") hide
         (effects (font (size 1 1) (thickness 0.15)))
     )

Commit message: CAN 1.85 rev 7: LC filter on the display's supply, JST XH for J1
Rev 6 in the car: the display's touch needed a hard press. A second LC
stage after the regulator (L2 1 uH, C9 C10 22 uF, C11 100 nF), its
corner about 30 kHz, keeps the 2.1 MHz ripple some 70 dB lower off the
display; the feedback stays before it. L2 about 12 mm from L1.

J1 is a JST XH 2.5 mm (B4B-XH-A, C144395, through hole): bigger crimps
than the PH, ready-made leads. The T5 vent's lid has its window moved
and grown for it. Readable schematic: D1 and D3 named as fitted.

Co-Authored-By: Claude Opus 5.5 <noreply@anthropic.com>
Claude-Session: https://claude.ai/code/session_018SKN4tJhAPpVCWtvRZgZpD
Parts:
- added C10: 22u 16V, Capacitor_SMD:C_1206_3216Metric, F.Cu at (149.1, 115.9)
- added C11: 100n, Capacitor_SMD:C_0603_1608Metric, F.Cu at (153.0, 116.2)
- added C9: 22u 16V, Capacitor_SMD:C_1206_3216Metric, F.Cu at (144.4, 116.0)
- added L2: 1u, Inductor_SMD:L_Sunlord_SWPA4026S, F.Cu at (150.5, 112.4)
- J1: footprint Connector_JST:JST_PH_B4B-PH-SM4-TB_1x04-1MP_P2.00mm_Vertical -> Connector_JST:JST_XH_B4B-XH-A_1x04_P2.50mm_Vertical
- moved J1 3.78 mm to (148.2, 84.0)
Connections:
- J3 pad 1: BAT_LCD -> BAT_OUT
Routing:
- net +3V3: track 50.9 -> 28.8 mm
- net BAT_OUT: track 0.00 -> 20.1 mm
- net TMID: track 18.9 -> 9.61 mm, vias 2 -> 0
- net FB: track 5.60 -> 12.9 mm, vias 0 -> 2
- net CANL: track 40.9 -> 35.2 mm
- net BAT_LCD: track 30.4 -> 27.9 mm
- net GND: track 157.8 -> 156.3 mm, vias 77 -> 80
- net CANH: track 35.3 -> 36.1 mm, vias 0 -> 2
- net TXD: track 18.5 -> 19.2 mm, vias 0 -> 1
Other:
- board text added: "rev 7"
- board text removed: "rev 6"
